File: power.kicad_sch (KiCad schematic)
At the start: 5 parts, among them U301 MCP1754ST-3302E/MB

Commit message: bom
Parts:
- C301, C303: MPN (none) -> C440198
- U301: MPN (none) -> C632035
Changed lines of the file:
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@@
+			)
+		)
+		(property "MPN" "C632035"
+			(at 143.51 95.25 0)
+			(effects
+				(font
+					(size 1.524 1.524)
+				)
+				(hide yes)
 			)
 		)
@@
 			)
 		)
+		(property "MPN" "C440198"
+			(at 129.54 100.33 0)
+			(effects
+				(font
+					(size 1.524 1.524)
+				)
+				(hide yes)
+			)
+		)
 		(pin "2"
 		)
@@
 			)
 		)
+		(property "MPN" "C440198"
+			(at 156.21 100.33 0)
+			(effects
+				(font
+					(size 1.524 1.524)
+				)
+				(hide yes)
+			)
+		)
