File: connectors.kicad_sch (KiCad schematic)
At the start: 3 parts, among them P501 USB_OTG, X501 CON_SWD, X502 SUB-D9

Commit message: bom
Parts:
- P501: MPN (none) -> C505245
Changed lines of the file:
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@@
+			)
+		)
+		(property "MPN" "C505245"
+			(at 109.22 78.74 0)
+			(effects
+				(font
+					(size 1.524 1.524)
+				)
+				(hide yes)
 			)
 		)

Commit message: usb-c
Parts:
- removed P501: USB_OTG, usb:Molex-Micro-USB-B-Middle-Mount, symbol candleLight-rescue:USB_OTG
- added P1: USB_C_Plug_USB2.0, Connector_USB:USB_C_Receptacle_G-Switch_GT-USB-7010ASV, symbol Connector:USB_C_Plug_USB2.0
- added R1: 5k1, Resistor_SMD:R_0603_1608Metric, symbol Device:R
Connections:
- net +5V: now also P1.A4 (VBUS), P1.A9 (VBUS), P1.B4 (VBUS), P1.B9 (VBUS)
- net GND: now also P1.A1 (GND), P1.A12 (GND), P1.B1 (GND), P1.B12 (GND), P1.S1 (SHIELD), R1.1
- net USB_DP: now also P1.A6 (D+)
- new net: P1.A5 (CC), R1.2
- new net USB_DN: P1.A7 (D-)
