File: mcu.kicad_sch (KiCad schematic)
At the start: 22 parts, among them U201 STM32F072C8Tx, Y201 8MHz

Commit message: bom
Parts:
- C201, C202: MPN (none) -> C91702
- C203, C204, C205, C206: MPN (none) -> C14663
- C207: MPN (none) -> C440198
- C208: MPN (none) -> C105621
- R201, R202: MPN (none) -> C23162
- R204: MPN (none) -> C21190
- U201: MPN (none) -> C80488
- Y201: MPN (none) -> C144380
Changed lines of the file:
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@@
+			)
+		)
+		(property "MPN" "C80488"
+			(at 147.32 99.06 0)
+			(effects
+				(font
+					(size 1.524 1.524)
+				)
+				(hide yes)
 			)
 		)
@@
 			)
 		)
+		(property "MPN" "C144380"
+			(at 34.29 80.01 0)
+			(effects
+				(font
+					(size 1.524 1.524)
+				)
+				(hide yes)
+			)
+		)
 		(pin "1"
 		)
@@
 			)
 		)
+		(property "MPN" "C23162"
+			(at 29.21 111.76 90)
+			(effects
+				(font
+					(size 1.524 1.524)
+				)
+				(hide yes)
+			)
+		)
 		(pin "2"
 		)
@@
 			)
 		)
+		(property "MPN" "C23162"
+			(at 29.21 114.3 90)
+			(effects
+				(font
+					(size 1.524 1.524)
+				)
+				(hide yes)
+			)
+		)
 		(pin "1"
 		)
@@
 			)
 		)
+		(property "MPN" "C21190"
+			(at 99.06 175.26 90)
+			(effects
+				(font
+					(size 1.524 1.524)
+				)
+				(hide yes)
+			)
+		)
 		(pin "1"
 		)
@@
 			)
 		)
+		(property "MPN" "C91702"
+			(at 27.94 77.47 90)
+			(effects
+				(font
+					(size 1.524 1.524)
+				)
+				(hide yes)
+			)
+		)
 		(pin "1"
 		)
@@
 			)
 		)
+		(property "MPN" "C91702"
+			(at 27.94 82.55 90)
+			(effects
+				(font
+					(size 1.524 1.524)
+				)
+				(hide yes)
+			)
+		)
 		(pin "2"
 		)
@@
 			)
 		)
+		(property "MPN" "C14663"
+			(at 63.5 173.99 0)
+			(effects
+				(font
+					(size 1.524 1.524)
+				)
+				(hide yes)
+			)
+		)
 		(pin "2"
 		)
@@
 			)
 		)
+		(property "MPN" "C14663"
+			(at 55.88 173.99 0)
+			(effects
+				(font
+					(size 1.524 1.524)
+				)
+				(hide yes)
+			)
+		)
 		(pin "1"
 		)
@@
 			)
 		)
+		(property "MPN" "C14663"
+			(at 48.26 173.99 0)
+			(effects
+				(font
+					(size 1.524 1.524)
+				)
+				(hide yes)
+			)
+		)
 		(pin "1"
 		)
@@
 			)
 		)
+		(property "MPN" "C14663"
+			(at 40.64 173.99 0)
+			(effects
+				(font
+					(size 1.524 1.524)
+				)
+				(hide yes)
+			)
+		)
 		(pin "1"
 		)
@@
 			)
 		)
+		(property "MPN" "C440198 "
+			(at 74.93 173.99 0)
+			(effects
+				(font
+					(size 1.524 1.524)
+				)
+				(hide yes)
+			)
+		)
 		(pin "1"
 		)
@@
 			)
 		)
+		(property "MPN" "C105621"
+			(at 34.29 67.31 0)
+			(effects
+				(font
+					(size 1.524 1.524)
+				)
+				(hide yes)
+			)
+		)

Commit message: usb-c
Connections:
- net USB_DM renamed USB_DN
Changed lines of the file:
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@@
 	(wire
 		(pts
-			(xy 245.11 124.46) (xy 243.84 124.46)
+			(xy 243.84 124.46) (xy 245.11 124.46)
 		)
 		(stroke
@@
 	(wire
 		(pts
-			(xy 245.11 127) (xy 243.84 127)
+			(xy 243.84 127) (xy 245.11 127)
 		)
 		(stroke
@@
 			)
 			(justify left bottom)
+		)
+	)
+	(global_label "USB_DN"
+		(shape input)
+		(at 245.11 124.46 0)
+		(fields_autoplaced yes)
+		(effects
+			(font
+				(size 1.524 1.524)
+			)
+			(justify left)
+		)
+		(property "Intersheetrefs" "${INTERSHEET_REFS}"
+			(at 256.7605 124.46 0)
+			(effects
+				(font
+					(size 1.27 1.27)
+				)
+				(justify left)
+				(hide yes)
+			)
+		)
+	)
+	(global_label "USB_DP"
+		(shape input)
+		(at 245.11 127 0)
+		(fields_autoplaced yes)
+		(effects
+			(font
+				(size 1.524 1.524)
+			)
+			(justify left)
+		)
+		(property "Intersheetrefs" "${INTERSHEET_REFS}"
+			(at 256.6879 127 0)
+			(effects
+				(font
+					(size 1.27 1.27)
+				)
+				(justify left)
+				(hide yes)
+			)
 		)
 	)
@@
 		)
 	)
-	(hierarchical_label "USB_DM"
-		(shape bidirectional)
-		(at 245.11 124.46 0)
-		(effects
-			(font
-				(size 1.524 1.524)
-			)
-			(justify left)
-		)
-	)
 	(hierarchical_label "LED2"
 		(shape output)
@@
 		(effects
 			(font
-				(size 1.524 1.524)
-			)
-			(justify left)
-		)
-	)
-	(hierarchical_label "USB_DP"
-		(shape bidirectional)
-		(at 245.11 127 0)
-		(effects
-			(font
