File: CAN.kicad_sch (KiCad schematic)
At the start: 5 parts, among them U401 TJA1051/3

Commit message: bom
Parts:
- C402, C403: MPN (none) -> C14663
- R401: MPN (none) -> C25804
- U401: MPN (none) -> C51484082
Changed lines of the file:
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@@
+			)
+		)
+		(property "MPN" "C51484082"
+			(at 146.05 91.44 0)
+			(effects
+				(font
+					(size 1.524 1.524)
+				)
+				(hide yes)
 			)
 		)
@@
 			)
 		)
+		(property "MPN" "C14663"
+			(at 152.4 118.11 0)
+			(effects
+				(font
+					(size 1.524 1.524)
+				)
+				(hide yes)
+			)
+		)
 		(pin "1"
 		)
@@
 			)
 		)
+		(property "MPN" "C14663"
+			(at 144.78 118.11 0)
+			(effects
+				(font
+					(size 1.524 1.524)
+				)
+				(hide yes)
+			)
+		)
 		(pin "2"
 		)
@@
 			)
 		)
+		(property "MPN" "C25804"
+			(at 115.57 78.74 90)
+			(effects
+				(font
+					(size 1.524 1.524)
+				)
+				(hide yes)
+			)
+		)

Commit message: schematic
Parts:
- removed C402, C403: 100nF, Capacitor_SMD:C_0603_1608Metric, symbol candleLight-rescue:C_Small
- removed R401: 10K, Resistor_SMD:R_0603_1608Metric, symbol candleLight-rescue:R
- removed R402: dnp, Resistor_SMD:R_0805_2012Metric, symbol candleLight-rescue:R
- removed U401: TJA1051/3, Package_SO:SOIC-8_3.9x4.9mm_P1.27mm, symbol candleLight-rescue:TJA1051/3
