File: candleLight.kicad_pcb (KiCad board)
At the start: 2 copper layers, 37.7 x 20 mm, 44 parts, among them P501 USB_OTG, U201 STM32F072C8Tx, U301 MCP1754ST-3302E/MB, U401 TJA1051/3, X501 CON_SWD, X502 SUB-D9, Y201 8MHz

Commit message: kicad 9
Parts:
- C201, C202, C203, C204, C205, C206, C208, C402, C403: footprint Capacitors_SMD:C_0603 -> Capacitor_SMD:C_0603_1608Metric
- C207, C301, C303: footprint Capacitors_SMD:C_0805 -> Capacitor_SMD:C_0805_2012Metric
- D601, D602, D603: footprint LEDs:LED_0603 -> LED_SMD:LED_0603_1608Metric
- R201, R202, R204, R401, R601, R602, R603: footprint Resistors_SMD:R_0603 -> Resistor_SMD:R_0603_1608Metric
- R203, R402: footprint Resistors_SMD:R_0805 -> Resistor_SMD:R_0805_2012Metric
- U201: footprint Housings_QFP:LQFP-48_7x7mm_Pitch0.5mm -> Package_QFP:LQFP-48_7x7mm_P0.5mm
- U301: footprint TO_SOT_Packages_SMD:SOT89-3_Housing -> Package_TO_SOT_SMD:SOT-89-3
- U401: footprint Housings_SOIC:SOIC-8_3.9x4.9mm_Pitch1.27mm -> Package_SO:SOIC-8_3.9x4.9mm_P1.27mm
- X501: footprint tagconnect:TC2030-NL -> Connector:Tag-Connect_TC2030-IDC-NL_2x03_P1.27mm_Vertical
- Y201: footprint Crystals:ABM3 -> Crystal:Crystal_SMD_Abracon_ABM3-2Pin_5.0x3.2mm
- moved U301 0.34 mm to (66.7, 79.1), turned to 180 degrees
- renumbered TX to W201, RX to W202, SCL to W203, SDA to W204, CS to W205, SCK to W206, MISO to W207, MOSI to W208
Connections:
- net /MCU/CAN_RX renamed /CAN/CAN_RXD
- net /MCU/CAN_TX renamed /CAN/CAN_TXD
- P501 pad 4: (no net) -> unconnected-(P501-ID-Pad4)
- U201 pad 12: (no net) -> unconnected-(U201-ADC_IN2/COMP2_INM/COMP2_OUT/SYS_WKUP4/TIM15_CH1/TIM2_CH3/TSC_G1_IO3/USART2_TX/PA2-Pad12)
- U201 pad 13: (no net) -> unconnected-(U201-ADC_IN3/COMP2_INP/TIM15_CH2/TIM2_CH4/TSC_G1_IO4/USART2_RX/PA3-Pad13)
- U201 pad 14: (no net) -> unconnected-(U201-ADC_IN4/COMP1_INM/COMP2_INM/DAC_OUT1/I2S1_WS/SPI1_NSS/TIM14_CH1/TSC_G2_IO1/USART2_CK/PA4-Pad14)
- U201 pad 15: (no net) -> unconnected-(U201-ADC_IN5/CEC/COMP1_INM/COMP2_INM/DAC_OUT2/I2S1_CK/SPI1_SCK/TIM2_CH1/TIM2_ETR/TSC_G2_IO2/PA5-Pad15)
- U201 pad 16: (no net) -> unconnected-(U201-ADC_IN6/COMP1_OUT/I2S1_MCK/SPI1_MISO/TIM16_CH1/TIM1_BKIN/TIM3_CH1/TSC_G2_IO3/USART3_CTS/PA6-Pad16)
- U201 pad 17: (no net) -> unconnected-(U201-ADC_IN7/COMP2_OUT/I2S1_SD/SPI1_MOSI/TIM14_CH1/TIM17_CH1/TIM1_CH1N/TIM3_CH2/TSC_G2_IO4/PA7-Pad17)
- U201 pad 18: (no net) -> unconnected-(U201-PB0/ADC_IN8/TIM1_CH2N/TIM3_CH3/TSC_G3_IO2/USART3_CK-Pad18)
- U201 pad 19: (no net) -> unconnected-(U201-PB1/ADC_IN9/TIM14_CH1/TIM1_CH3N/TIM3_CH4/TSC_G3_IO3/USART3_DE/USART3_RTS-Pad19)
- U201 pad 20: (no net) -> unconnected-(U201-PB2/TSC_G3_IO4-Pad20)
- U201 pad 21: (no net) -> unconnected-(U201-PB10/CEC/I2C2_SCL/I2S2_CK/SPI2_SCK/TIM2_CH3/TSC_SYNC/USART3_TX-Pad21)
- U201 pad 22: (no net) -> unconnected-(U201-PB11/I2C2_SDA/TIM2_CH4/TSC_G6_IO1/USART3_RX-Pad22)
- U201 pad 29: (no net) -> unconnected-(U201-CRS_SYNC/RCC_MCO/TIM1_CH1/USART1_CK/PA8-Pad29)
- U201 pad 3: (no net) -> unconnected-(U201-PC14/RCC_OSC32_IN-Pad3)
- U201 pad 38: (no net) -> unconnected-(U201-I2S1_WS/SPI1_NSS/TIM2_CH1/TIM2_ETR/USART2_RX/USART4_DE/USART4_RTS/PA15-Pad38)
- U201 pad 39: (no net) -> unconnected-(U201-PB3/I2S1_CK/SPI1_SCK/TIM2_CH2/TSC_G5_IO1-Pad39)
- U201 pad 4: (no net) -> unconnected-(U201-PC15/RCC_OSC32_OUT-Pad4)
- U201 pad 40: (no net) -> unconnected-(U201-PB4/I2S1_MCK/SPI1_MISO/TIM17_BKIN/TIM3_CH1/TSC_G5_IO2-Pad40)
- U201 pad 41: (no net) -> unconnected-(U201-PB5/I2C1_SMBA/I2S1_SD/SPI1_MOSI/SYS_WKUP6/TIM16_BKIN/TIM3_CH2-Pad41)
- X501 pad 6: (no net) -> unconnected-(X501-SWO-Pad6)
- X502 pad 1: (no net) -> unconnected-(X502-Pad1)
- X502 pad 4: (no net) -> unconnected-(X502-Pad4)
- X502 pad 5: (no net) -> unconnected-(X502-Pad5)
- X502 pad 6: (no net) -> unconnected-(X502-Pad6)
- X502 pad 8: (no net) -> unconnected-(X502-Pad8)
- X502 pad 9: (no net) -> unconnected-(X502-Pad9)
Routing:
- net (no net): track 3.10 -> 0.00 mm
- net GND: track 148.8 -> 147.1 mm
- net +3V3: track 117.3 -> 116.6 mm, vias 4 -> 2
- net /CAN/CAN_S: track 18.2 -> 18.8 mm
Other:
- net class Default removed
- board text added: "candleLight"
- board text removed: "candleLight v1.1"
- board text removed: "http://bytewerk.org"

Commit message: bom
Parts:
- added G***: LOGO, LOGO, B.Cu at (64.1, 83.7)
- moved C207 0.30 mm to (61.1, 93.0)
- moved C402 0.17 mm to (62.9, 93.2)
- moved C206 0.15 mm to (59.3, 93.2)
- moved R203 0.10 mm to (57.6, 93.0)
- renumbered W206 to CHK, W205 to CS, W207 to MISO, W208 to MOSI, W202 to RX, W203 to SCL, W204 to SDA, W201 to TX
Routing:
- net /CAN/CAN_TXD: track 8.98 -> 7.95 mm
Other:
- board text added: "CANH"
- board text added: "CANL"
- board text removed: "CAN_H"
- board text removed: "candleLight"

Commit message: usb-c
Parts:
- removed FID101, FID102, FID103: Dummy_FIDUCIAL_Passermarke_Type1_RevE_Date16Nov2011, Fiducials:Fiducial_1mm_Dia_2.54mm_Outer_CopperTop
- removed P501: USB_OTG, usb:Molex-Micro-USB-B-Middle-Mount
- added P1: USB_C_Plug_USB2.0, Connector_USB:USB_C_Receptacle_G-Switch_GT-USB-7010ASV, F.Cu at (44.5, 84.7)
- added R1: 5k1, Resistor_SMD:R_0603_1608Metric, F.Cu at (45.1, 77.7)
- moved W301 1.01 mm to (48.3, 77.5)
- moved W302 1.00 mm to (44.3, 77.5)
- moved C205 0.10 mm to (52.4, 77.7)
- renumbered TX to W201, RX to W202, SCL to W203, SDA to W204, CS to W205, CHK to W206, MISO to W207, MOSI to W208
Connections:
- U201 pad 32: /Connectors/USB_DM -> USB_DN
- U201 pad 33: /Connectors/USB_DP -> USB_DP
Routing:
- net +3V3: track 116.7 -> 5.57 mm
- net GND: track 147.3 -> 54.9 mm, vias 24 -> 28
- net Net-(P1-CC): track 0.00 -> 6.73 mm
- net +5V: track 58.4 -> 64.9 mm, vias 4 -> 5
- net USB_DN: track 0.00 -> 6.16 mm, vias 0 -> 2
- net USB_DP: track 0.00 -> 5.79 mm
- net /Connectors/USB_DM: track 5.79 -> 0.00 mm
- net /Connectors/USB_DP: track 5.73 -> 0.00 mm
Other:
- board size 37.7 x 20 mm -> 38.8 x 20 mm

Commit message: schematic
Parts:
- removed P1: USB_C_Plug_USB2.0, Connector_USB:USB_C_Receptacle_G-Switch_GT-USB-7010ASV
- removed the R1 at (45.1, 77.7)
- added J1: USB_C_Receptacle_USB2.0, stm32world:USB_C_Receptacle_HRO_TYPE-C-31-M-12, F.Cu at (44.1, 84.8)
- added R11: 5k1, Resistor_SMD:R_0603_1608Metric, F.Cu at (47.8, 77.6)
- added R5: 5k1, Resistor_SMD:R_0603_1608Metric, F.Cu at (49.3, 77.6)
- SCL1: renamed from W203; value TEST_1P -> SCL1
- SDA1: renamed from W204; value TEST_1P -> SDA1
- U1: renamed from U301; value MCP1754ST-3302E/MB -> ME6210A33PG
- moved G*** 1.20 mm to (64.1, 84.9)
- moved C12 0.12 mm to (72.4, 93.2)
- renumbered C301 to C1, C207 to C10, C402 to C11, C403 to C12, C303 to C2, C201 to C3, C202 to C4, C208 to C5, C203 to C6, C204 to C7, C205 to C8, C206 to C9, D601 to D1, D602 to D2, D603 to D3, R201 to R1, R603 to R10, R202 to R2, R203 to R3, R204 to R4, R401 to R6, R402 to R7, R601 to R8, R602 to R9, U201 to U2, U401 to U3, W301 to W1, W302 to W2, W205 to W3, W206 to W4, W207 to W5, W208 to W6, W201 to W7, W202 to W8, X501 to X1, X502 to X2, Y201 to Y1
Connections:
- net /CAN/CAN_H renamed CAN_H
- net /CAN/CAN_L renamed CAN_L
- net /CAN/CAN_RXD renamed CAN_RX
- net /CAN/CAN_S renamed /CAN_S
- net /CAN/CAN_TXD renamed CAN_TX
- net /Connectors/NRST renamed NRST
- net /Connectors/SWCLK renamed SWCLK
- net /Connectors/SWDIO renamed SWDIO
- net /LEDs/LED1 renamed LED1
- net /LEDs/LED2 renamed LED2
- net /MCU/BOOT0 renamed Net-(U2-BOOT0)
- U1 pad 1: +5V -> GND
- U1 pad 2: GND -> +5V
Routing:
- net Net-(J1-CC2): track 0.00 -> 10.7 mm
- net GND: track 54.9 -> 47.9 mm, vias 28 -> 20
- net Net-(P1-CC): track 6.73 -> 0.00 mm
- net Net-(J1-CC1): track 0.00 -> 5.97 mm
- net +5V: track 64.9 -> 67.4 mm
- net USB_DP: track 5.79 -> 8.18 mm
- net USB_DN: track 6.16 -> 8.20 mm, vias 2 -> 0
- net +3V3: track 5.57 -> 7.59 mm, vias 2 -> 4
- net Net-(U2-PA10): track 4.60 -> 3.33 mm
- net Net-(U2-PA9): track 3.17 -> 2.44 mm
Other:
- board size 38.8 x 20 mm -> 39.1 x 20 mm

Commit message: v2 ready
Parts:
- removed X1: CON_SWD, Connector:Tag-Connect_TC2030-IDC-NL_2x03_P1.27mm_Vertical
- removed X2: SUB-D9, subd9:DB9M_CI
- added J2: Conn_Phoenix, TerminalBlock_Phoenix:TerminalBlock_Phoenix_MKDS-1,5-3-5.08_1x03_P5.08mm_Horizontal, F.Cu at (80.8, 90.3)
- added J3: Conn_SWD, Connector_PinHeader_2.54mm:PinHeader_1x03_P2.54mm_Vertical, F.Cu at (47.3, 92.5)
- added J4: Conn_3.3V, Connector_PinHeader_2.54mm:PinHeader_1x02_P2.54mm_Vertical, F.Cu at (42.2, 77.2)
- moved W2 31.9 mm to (76.2, 77.3)
- moved W1 24.1 mm to (72.3, 77.3)
- moved G*** 5.80 mm to (69.9, 85.1)
- moved C12 0.50 mm to (72.9, 93.2)
- moved R6 0.40 mm to (74.4, 93.2)
Connections:
- net /CAN_S renamed CAN_S
Routing:
- net GND: track 47.9 -> 38.6 mm
- net CAN_H: track 15.2 -> 20.2 mm, vias 1 -> 0
- net CAN_L: track 13.9 -> 18.5 mm
- net NRST: track 23.7 -> 20.2 mm, vias 4 -> 3
- net SWCLK: track 11.3 -> 13.4 mm
- net SWDIO: track 12.8 -> 14.5 mm
- net +5V: track 67.4 -> 66.5 mm
- net Net-(J1-CC2): track 10.7 -> 11.2 mm
Other:
- board size 39.1 x 20 mm -> 46.4 x 20 mm
- board text added: "3V3"
- board text added: "CAN_H"
- board text added: "CAN_L"
- board text added: "CLK"
- board text added: "CS"
- board text added: "IO"
- board text added: "MISO"
- board text added: "MOSI"
- board text added: "RST"
- board text added: "SCK"
- board text added: "SCL"
- board text added: "SDA"
- board text removed: "CANH"
- board text removed: "CANL"

Commit message: production :)
Parts:
- C3, C4: value 20pF -> 30pF
Changed lines of the file:
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@@
 			)
 		)
-		(property "Value" "20pF"
+		(property "Value" "30pF"
 			(at 0 1.43 180)
 			(layer "F.Fab")
@@
 			)
 		)
-		(property "MPN" "C1648"
+		(property "MPN" "C1658"
 			(at 0 0 180)
 			(unlocked yes)
@@
 			)
 		)
-		(property "Value" "20pF"
+		(property "Value" "30pF"
 			(at 0 1.43 180)
 			(layer "F.Fab")
@@
 			)
 		)
-		(property "MPN" "C1648"
+		(property "MPN" "C1658"
 			(at 0 0 180)
 			(unlocked yes)
@@
 			)
 		)
-		(property "MPN" "C51484082"
+		(property "MPN" "C58988"
 			(at 0 0 0)
 			(unlocked yes)

Commit message: update schematic
Parts:
- R3: value R -> dnp
